File: kicad/rosalyn-fc.kicad_pcb (KiCad board)
At the start: 4 copper layers, 40 x 40 mm, 58 parts, among them J1 USB-C, J10 Buzzer, J11 PWM_LED, J2 GPS/MAG, J3 Terminal, J4 Satellite, J5 Serial1, J6 Serial2, J7 ESC, J8 SWD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

Commit message: ready for review
Parts:
- removed J10: Buzzer, Connector_PinHeader_2.54mm:PinHeader_1x02_P2.54mm_Vertical
- removed J11: PWM_LED, Connector_PinHeader_2.54mm:PinHeader_1x03_P2.54mm_Vertical
- removed J8: SWD, rosalyn-fc:JST_SH_SM04B-SRSS-TB_1x04-1MP_P1.00mm_Horizontal
- removed J9: Expansion, Connector_PinHeader_2.54mm:PinHeader_1x08_P2.54mm_Vertical
- added SW1: Boot, rosalyn-fc:TACT-SWITCH, F.Cu at (142.3, 93.0)
- added TP1: buz+, TestPoint:TestPoint_Pad_1.5x1.5mm, F.Cu at (141.0, 86.4)
- added TP10: 5v, TestPoint:TestPoint_Pad_1.5x1.5mm, F.Cu at (158.9, 81.4)
- added TP11: gnd, TestPoint:TestPoint_Pad_1.5x1.5mm, F.Cu at (131.5, 97.4)
- added TP12: swclk, TestPoint:TestPoint_Pad_1.5x1.5mm, F.Cu at (131.5, 100.0)
- added TP13: swdio, TestPoint:TestPoint_Pad_1.5x1.5mm, F.Cu at (131.5, 102.5)
- added TP14: led-, TestPoint:TestPoint_Pad_1.5x1.5mm, F.Cu at (159.0, 118.5)
- added TP15: led+, TestPoint:TestPoint_Pad_1.5x1.5mm, F.Cu at (159.0, 115.9)
- added TP16: led_sig, TestPoint:TestPoint_Pad_1.5x1.5mm, F.Cu at (159.0, 113.4)
- added TP2: buz-, TestPoint:TestPoint_Pad_1.5x1.5mm, F.Cu at (141.0, 88.9)
- added TP3: M5, TestPoint:TestPoint_Pad_1.5x1.5mm, F.Cu at (141.1, 81.4)
- added TP4: M6, TestPoint:TestPoint_Pad_1.5x1.5mm, F.Cu at (143.7, 81.4)
- added TP5: PPM, TestPoint:TestPoint_Pad_1.5x1.5mm, F.Cu at (146.2, 81.4)
- added TP6: Camera, TestPoint:TestPoint_Pad_1.5x1.5mm, F.Cu at (148.8, 81.4)
- added TP7: rssi, TestPoint:TestPoint_Pad_1.5x1.5mm, F.Cu at (151.3, 81.4)
- added TP8: gnd, TestPoint:TestPoint_Pad_1.5x1.5mm, F.Cu at (153.8, 81.4)
- added TP9: 3v3, TestPoint:TestPoint_Pad_1.5x1.5mm, F.Cu at (156.4, 81.4)
- C6, C7: footprint Capacitor_SMD:C_0603_1608Metric -> Capacitor_SMD:C_0805_2012Metric
- D1: moved to B.Cu
- moved C8 2.94 mm to (148.2, 87.1), turned to 180 degrees
- moved D3 1.64 mm to (159.7, 105.1)
- moved R9 1.64 mm to (161.3, 105.0)
- moved FB1 0.47 mm to (146.4, 109.9)
- moved C6 0.33 mm to (144.5, 109.9)
- moved C7 0.21 mm to (138.7, 109.9)
Routing:
- net swclk: track 10.8 -> 14.4 mm
- net nrst: track 5.67 -> 9.18 mm
- net uart6_rxtx: track 34.3 -> 31.5 mm
- net +5V: track 112.2 -> 109.5 mm, vias 2 -> 4
- net m2: track 20.8 -> 23.2 mm
- net +3V3: track 34.8 -> 37.2 mm, vias 13 -> 12
- net swdio: track 15.6 -> 17.9 mm
- net boot0: track 8.12 -> 10.4 mm, vias 0 -> 1
- net m5: track 20.5 -> 22.6 mm
- net led0: track 9.47 -> 7.36 mm
- net m1: track 24.3 -> 26.2 mm
- net Net-(Q1-Pad2): track 2.97 -> 4.72 mm, vias 0 -> 1
- net Net-(D1-Pad2): track 15.3 -> 16.8 mm, vias 1 -> 0
- net camera: track 19.0 -> 20.4 mm, vias 2 -> 3
- net rssi_adc: track 12.5 -> 13.6 mm
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