File: kicad/rosalyn-fc.sch (KiCad schematic (older format))
At the start: 58 parts, among them J1 USB-C, J10 Buzzer, J11 PWM_LED, J2 GPS/MAG, J3 Terminal, J4 Satellite, J5 Serial1, J6 Serial2, J7 ESC, J8 SWD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

Commit message: ready for review
Parts:
- removed J10: Buzzer, Connector_PinHeader_2.54mm:PinHeader_1x02_P2.54mm_Vertical, symbol Connector_Generic:Conn_01x02
- removed J11: PWM_LED, Connector_PinHeader_2.54mm:PinHeader_1x03_P2.54mm_Vertical, symbol Connector_Generic:Conn_01x03
- removed J8: SWD, rosalyn-fc:JST_SH_SM04B-SRSS-TB_1x04-1MP_P1.00mm_Horizontal, symbol Connector_Generic:Conn_01x04
- removed J9: Expansion, Connector_PinHeader_2.54mm:PinHeader_1x08_P2.54mm_Vertical, symbol Connector_Generic:Conn_01x08
- added SW1: Boot, rosalyn-fc:TACT-SWITCH, symbol rosalyn-fc:TACT-SWITCH
- added TP1: buz+, TestPoint:TestPoint_Pad_1.5x1.5mm, symbol Connector:TestPoint
- added TP10: 5v, TestPoint:TestPoint_Pad_1.5x1.5mm, symbol Connector:TestPoint
- added TP11, TP8: gnd, TestPoint:TestPoint_Pad_1.5x1.5mm, symbol Connector:TestPoint
- added TP12: swclk, TestPoint:TestPoint_Pad_1.5x1.5mm, symbol Connector:TestPoint
- added TP13: swdio, TestPoint:TestPoint_Pad_1.5x1.5mm, symbol Connector:TestPoint
- added TP14: led-, TestPoint:TestPoint_Pad_1.5x1.5mm, symbol Connector:TestPoint
- added TP15: led+, TestPoint:TestPoint_Pad_1.5x1.5mm, symbol Connector:TestPoint
- added TP16: led_sig, TestPoint:TestPoint_Pad_1.5x1.5mm, symbol Connector:TestPoint
- added TP2: buz-, TestPoint:TestPoint_Pad_1.5x1.5mm, symbol Connector:TestPoint
- added TP3: M5, TestPoint:TestPoint_Pad_1.5x1.5mm, symbol Connector:TestPoint
- added TP4: M6, TestPoint:TestPoint_Pad_1.5x1.5mm, symbol Connector:TestPoint
- added TP5: PPM, TestPoint:TestPoint_Pad_1.5x1.5mm, symbol Connector:TestPoint
- added TP6: Camera, TestPoint:TestPoint_Pad_1.5x1.5mm, symbol Connector:TestPoint
- added TP7: rssi, TestPoint:TestPoint_Pad_1.5x1.5mm, symbol Connector:TestPoint
- added TP9: 3v3, TestPoint:TestPoint_Pad_1.5x1.5mm, symbol Connector:TestPoint
- C6, C7: footprint Capacitor_SMD:C_0603_1608Metric -> Capacitor_SMD:C_0805_2012Metric
Connections:
- net +3V3: now also SW1.1, TP9.1
- net +5V: now also TP1.1, TP10.1, TP15.1
- net GND: now also TP11.1, TP14.1, TP8.1
- net boot0: now also SW1.2
- net camera: now also TP6.1
- net led: now also TP16.1
- net m5: now also TP3.1
- net m6: now also TP4.1
- net ppm: now also TP5.1
- net rssi_adc: now also TP7.1
- net swclk: now also TP12.1
- net swdio: now also TP13.1
- net at Q1.2 (C): now also TP2.1
- net max7456_cs renamed spi2_cs
Other:
- moved on the sheet: C1, C15, U2, U4, Y1
